File: KiCAD/OpenTRSwitch/OpenTRSwitch.kicad_sch (KiCad schematic)
At the start: 28 parts, among them X1 B12T-Logo

Commit message: added default diodes as comment
Other:
- company: (none) -> Bridge12Technologies
- title: (none) -> Passive TR Switch
Changed lines of the file:
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@@
 (kicad_sch (version 20230121) (generator eeschema)
   (paper "A4")
+  (title_block
+    (title "Passive TR Switch")
+    (date "2023-06-09")
+    (rev "1.0")
+    (company "Bridge12Technologies")
+    (comment 1 "DEFAULT SUGGESTED DIODES: 1N4148")
+  )
   (junction (at 82.55 47.244) (diameter 0) (color 0 0 0 0)
   )
